File: project/Power.sch (KiCad schematic (older format))
At the start: 26 parts, among them U1 TPS2115a, U2 TPS82740B, U3 MCP73831

Commit message: fix
Parts:
- BT1: symbol spora-rescue:BAT_CON -> template-rescue:BAT_CON
- C1, C2, C22, C3, C4, C5, C6, C7: symbol spora-rescue:C_Small -> template-rescue:C_Small
- D1: symbol spora-rescue:ZENER-RESCUE-versionA -> template-rescue:ZENER-RESCUE-versionA
- G2: symbol spora-rescue:LOGO_INTI -> template-rescue:LOGO_INTI
- R1, R15, R16, R17, R18, R2, R3, R4: symbol spora-rescue:R_Small -> template-rescue:R_Small
- TP1, TP2, TP3: symbol spora-rescue:TESTPOINT -> template-rescue:TESTPOINT
- U1: symbol spora-rescue:TPS2115a -> template-rescue:TPS2115a
- U2: symbol spora-rescue:TPS82740B -> template-rescue:TPS82740B
- U3: symbol spora-rescue:MCP73831 -> template-rescue:MCP73831
- USB1: symbol spora-rescue:USB-MINI -> template-rescue:USB-MINI
Changed lines of the file:
@@
 $EndDescr
 $Comp
-L spora-rescue:GND-RESCUE-versionA #PWR040
+L template-rescue:GND-RESCUE-versionA #PWR040
 U 1 1 587000D5
 P 6600 5100
@@
 $EndComp
 $Comp
-L spora-rescue:C_Small C4
+L template-rescue:C_Small C4
 U 1 1 587000E5
 P 8250 4550
@@
 $EndComp
 $Comp
-L spora-rescue:GND-RESCUE-versionA #PWR041
+L template-rescue:GND-RESCUE-versionA #PWR041
 U 1 1 587000EC
 P 8250 4700
@@
 $EndComp
 $Comp
-L spora-rescue:GND-RESCUE-versionA #PWR042
+L template-rescue:GND-RESCUE-versionA #PWR042
 U 1 1 587000FD
 P 6350 4700
@@
 $EndComp
 $Comp
-L spora-rescue:+3.3V-RESCUE-versionA #+3.3V043
+L template-rescue:+3.3V-RESCUE-versionA #+3.3V043
 U 1 1 58700103
 P 8950 4400
@@
 $EndComp
 $Comp
-L spora-rescue:GND-RESCUE-versionA #PWR044
+L template-rescue:GND-RESCUE-versionA #PWR044
 U 1 1 58700109
 P 4600 5250
@@
 $EndComp
 $Comp
-L spora-rescue:GND-RESCUE-versionA #PWR045
+L template-rescue:GND-RESCUE-versionA #PWR045
 U 1 1 5870010F
 P 5250 5250
@@
 $EndComp
 $Comp
-L spora-rescue:+VBAT #PWR046
+L template-rescue:+VBAT #PWR046
 U 1 1 58700115
 P 3500 4300
@@
 $EndComp
 $Comp
-L spora-rescue:C_Small C7
+L template-rescue:C_Small C7
 U 1 1 5870011F
 P 3750 5050
@@
 $EndComp
 $Comp
-L spora-rescue:GND-RESCUE-versionA #PWR047
+L template-rescue:GND-RESCUE-versionA #PWR047
 U 1 1 58700126
 P 3750 5250
@@
 $EndComp
 $Comp
-L spora-rescue:C_Small C6
+L template-rescue:C_Small C6
 U 1 1 58700130
 P 3500 5050
@@
 $EndComp
 $Comp
-L spora-rescue:GND-RESCUE-versionA #PWR048
+L template-rescue:GND-RESCUE-versionA #PWR048
 U 1 1 58700137
 P 3500 5250
@@
 $EndComp
 $Comp
-L spora-rescue:R_Small R4
+L template-rescue:R_Small R4
 U 1 1 58700141
 P 4000 5050
@@
 $EndComp
 $Comp
-L spora-rescue:GND-RESCUE-versionA #PWR049
+L template-rescue:GND-RESCUE-versionA #PWR049
 U 1 1 58700148
 P 4000 5250
@@
 $EndComp
 $Comp
-L spora-rescue:R_Small R1
+L template-rescue:R_Small R1
 U 1 1 58700152
 P 5300 4400
@@
 $EndComp
 $Comp
-L spora-rescue:TPS82740B U2
+L template-rescue:TPS82740B U2
 U 1 1 5870016E
 P 6700 4300
@@
 NoConn ~ 8100 4900
 $Comp
-L spora-rescue:USB-MINI USB1
+L template-rescue:USB-MINI USB1
 U 1 1 58700EDC
 P 3600 1950
@@
 $EndComp
 $Comp
-L spora-rescue:GND-RESCUE-versionA #PWR050
+L template-rescue:GND-RESCUE-versionA #PWR050
 U 1 1 58700EE3
 P 4000 2400
@@
 $EndComp
 $Comp
-L spora-rescue:C_Small C1
+L template-rescue:C_Small C1
 U 1 1 58700EED
 P 6050 1850
@@
 $EndComp
 $Comp
-L spora-rescue:GND-RESCUE-versionA #PWR051
+L template-rescue:GND-RESCUE-versionA #PWR051
 U 1 1 58700EF4
 P 6050 2250
@@
 $EndComp
 $Comp
-L spora-rescue:C_Small C2
+L template-rescue:C_Small C2
 U 1 1 58700EFE
 P 7850 1850
@@
 $EndComp
 $Comp
-L spora-rescue:GND-RESCUE-versionA #PWR052
+L template-rescue:GND-RESCUE-versionA #PWR052
 U 1 1 58700F05
 P 7850 2250
@@
 $EndComp
 $Comp
-L spora-rescue:R_Small R2
+L template-rescue:R_Small R2
 U 1 1 58700F0F
 P 7600 2050
@@
 $EndComp
 $Comp
-L spora-rescue:GND-RESCUE-versionA #PWR053
+L template-rescue:GND-RESCUE-versionA #PWR053
 U 1 1 58700F16
 P 7600 2250
@@
 $EndComp
 $Comp
-L spora-rescue:GND-RESCUE-versionA #PWR054
+L template-rescue:GND-RESCUE-versionA #PWR054
 U 1 1 58700F1C
 P 7450 2250
@@
 $EndComp
 $Comp
-L spora-rescue:ZENER-RESCUE-versionA D1
+L template-rescue:ZENER-RESCUE-versionA D1
 U 1 1 58700F26
 P 4200 2100
@@
 $EndComp
 $Comp
-L spora-rescue:GND-RESCUE-versionA #PWR055
+L template-rescue:GND-RESCUE-versionA #PWR055
 U 1 1 58700F2D
 P 4200 2400
@@
 $EndComp
 $Comp
-L spora-rescue:GND-RESCUE-versionA #PWR056
+L template-rescue:GND-RESCUE-versionA #PWR056
 U 1 1 58700F33
 P 3550 2600
@@
 $EndComp
 $Comp
-L spora-rescue:GND-RESCUE-versionA #PWR057
+L template-rescue:GND-RESCUE-versionA #PWR057
 U 1 1 58700F39
 P 3950 1450
@@
 $EndComp
 $Comp
-L spora-rescue:PWR_FLAG #FLG058
+L template-rescue:PWR_FLAG #FLG058
 U 1 1 58700F3F
 P 4150 1600
@@
 $EndComp
 $Comp
-L spora-rescue:GND-RESCUE-versionA #PWR059
+L template-rescue:GND-RESCUE-versionA #PWR059
 U 1 1 58700F45
 P 8200 2250
@@
 $EndComp
 $Comp
-L spora-rescue:+VBAT #PWR060
+L template-rescue:+VBAT #PWR060
 U 1 1 58700F4B
 P 8050 1450
@@
 $EndComp
 $Comp
-L spora-rescue:BAT_CON BT1
+L template-rescue:BAT_CON BT1
 U 1 1 58700F51
 P 8400 1650
@@
 $EndComp
 $Comp
-L spora-rescue:R_Small R3
+L template-rescue:R_Small R3
 U 1 1 58700F5C
 P 5850 2100
@@
 $EndComp
 $Comp
-L spora-rescue:C_Small C5
+L template-rescue:C_Small C5
 U 1 1 58700F67
 P 4500 2100
@@
 $EndComp
 $Comp
-L spora-rescue:MCP73831 U?
+L template-rescue:MCP73831 U?
 U 1 1 58700F72
 P 6850 1800
@@
 $EndComp
 $Comp
-L spora-rescue:GND-RESCUE-versionA #PWR061
+L template-rescue:GND-RESCUE-versionA #PWR061
 U 1 1 58700F79
 P 6900 2500
@@
 $EndComp
 $Comp
-L spora-rescue:GND-RESCUE-versionA #PWR062
+L template-rescue:GND-RESCUE-versionA #PWR062
 U 1 1 58700F7F
 P 4500 2400
@@
 $EndComp
 $Comp
-L spora-rescue:+3.3V-RESCUE-versionA #+3.3V063
+L template-rescue:+3.3V-RESCUE-versionA #+3.3V063
 U 1 1 58700F85
 P 5600 2050
@@
 Para calcular  ILIM se utiliza R4. \nSegún la hoja de datos recomienda que no se deje en cero, ver \nver página nº 17 (CURRENT LIMITING).\n500 / 1,5k = 333 mA\n
 $Comp
-L spora-rescue:LOGO_INTI G2
+L template-rescue:LOGO_INTI G2
 U 1 1 5873D882
 P 7950 6150
@@
 $EndBitmap
 $Comp
-L spora-rescue:R_Small R15
+L template-rescue:R_Small R15
 U 1 1 58793D3D
 P 2800 4500
@@
 $EndComp
 $Comp
-L spora-rescue:R_Small R17
+L template-rescue:R_Small R17
 U 1 1 58793DE0
 P 2800 4900
@@
 $EndComp
 $Comp
-L spora-rescue:GND-RESCUE-versionA #PWR064
+L template-rescue:GND-RESCUE-versionA #PWR064
 U 1 1 58793EE5
 P 2800 5250
@@
 $EndComp
 $Comp
-L spora-rescue:+VBAT #PWR065
+L template-rescue:+VBAT #PWR065
 U 1 1 58793F1F
 P 2800 4300
@@
 Connection ~ 2800 4650
 $Comp
-L spora-rescue:R_Small R16
+L template-rescue:R_Small R16
 U 1 1 587944FD
 P 3200 4500
@@
 $EndComp
 $Comp
-L spora-rescue:R_Small R18
+L template-rescue:R_Small R18
 U 1 1 58794503
 P 3200 4900
@@
 $EndComp
 $Comp
-L spora-rescue:GND-RESCUE-versionA #PWR066
+L template-rescue:GND-RESCUE-versionA #PWR066
 U 1 1 58794509
 P 3200 5250
@@
 $EndComp
 $Comp
-L spora-rescue:+VBAT #PWR067
+L template-rescue:+VBAT #PWR067
 U 1 1 5879450F
 P 3200 4300
@@
 STAT
 $Comp
-L spora-rescue:TPS2115a U1
+L template-rescue:TPS2115a U1
 U 1 1 587D5F1C
 P 4000 4250
@@
 	3500 4450 4000 4450
 $Comp
-L spora-rescue:C_Small C22
+L template-rescue:C_Small C22
 U 1 1 58B804E6
 P 8700 4550
@@
 $EndComp
 $Comp
-L spora-rescue:GND-RESCUE-versionA #PWR068
+L template-rescue:GND-RESCUE-versionA #PWR068
 U 1 1 58B806B8
 P 8700 4700
@@
 VCC
 $Comp
-L spora-rescue:C_Small C3
+L template-rescue:C_Small C3
 U 1 1 58B9B9CE
 P 6350 4550
@@
 	8200 2250 8200 1700
 $Comp
-L spora-rescue:TESTPOINT TP1
+L template-rescue:TESTPOINT TP1
 U 1 1 58BF3F88
 P 5200 1500
@@
 Connection ~ 5200 1600
 $Comp
-L spora-rescue:TESTPOINT TP2
+L template-rescue:TESTPOINT TP2
 U 1 1 58BF4215
 P 6000 4200
@@
 $EndComp
 $Comp
-L spora-rescue:TESTPOINT TP3
+L template-rescue:TESTPOINT TP3
 U 1 1 58BF4354
 P 8500 4250
