File: project/Power.sch (KiCad schematic (older format))
At the start: 26 parts, among them U1 TPS2115a, U2 TPS82740B, U3 MCP73831

Commit message: upate
Parts:
- removed G2: LOGO_INTI, symbol template-rescue:LOGO_INTI
